Commit message: V0.4.0 First complete version of 3d model and urdf

File: SkyGrip_URDF/urdf/SkyGrip_URDF.urdf (robot description, URDF)
Before this commit: robot mppi, 3 links, 2 joints
Links:
- link Link_1: mass 0.067836 -> 0.08; geometry collision mesh filename=package://SkyGrip_URDF/meshes/Link_1.STL; visual mesh filename=package://SkyGrip_URDF/meshes/Link_1.STL
- link Link_2: mass 0.031109 -> 0.105; geometry collision mesh filename=package://SkyGrip_URDF/meshes/Link_2.STL; visual mesh filename=package://SkyGrip_URDF/meshes/Link_2.STL
- link base_link: mass 1.1619 -> 1; geometry collision mesh filename=package://SkyGrip_URDF/meshes/base_link.STL; visual mesh filename=package://SkyGrip_URDF/meshes/base_link.STL
Joints:
- joint Joint_1: origin xyz=0.076125 -0.042332 -0.059398 rpy=-0.0039907 0 0 -> xyz=0.075884 -0.042123 -0.023898 rpy=-0.00065513 0 -0.0087266
- joint Joint_2: origin xyz=0 0 -0.1308 rpy=3.1379 0 0 -> xyz=0 0 -0.1308 rpy=-3.1379 0 0
